Commit message: feat(software): Set up RL training framework with corrected URDF model
Complete Phase 1 of the RL development plan: port the agibot_x1_train
IsaacGym training framework to Asimov v1, with a working 12-DOF
lower-body standing task configuration. Also fix two URDF conversion
bugs that caused link meshes to render in wrong positions.

Rewrite the MJCF→URDF converter to parse source XML directly instead
of going through MuJoCo's compiled model. Fixes two bugs:

1. Mesh placement: `mujoco.MjModel.from_xml_path()` silently shifts
   mesh geom positions to the mesh's center of mass for internal
   inertia accounting. URDF has no equivalent compensation, so meshes
   were placed at COM offsets. Links with mesh COMs far from origin
   (waist, hip, neck) rendered out of view, appearing "missing" in
   IsaacGym.

2. Inertial representation: previously emitted non-zero
   `<inertial><origin rpy>` with `ixx/iyy/izz` as principal-axis
   diagonals. While valid per URDF spec, many physics engines
   (IsaacGym included) ignore the inertial RPY and treat the
   diagonals as body-frame components.

Fixes:
- Parse MJCF as raw XML; copy body/geom pos/quat verbatim
- Emit body-frame 6-component inertia (`ixx ixy ixz iyy iyz izz`)
  from MJCF `fullinertia`, with `<origin rpy="0 0 0">`
- Add `Defaults` class to resolve MJCF `<default class>` inheritance
- Capsule geoms with `fromto` correctly compute midpoint and axis
  rotation for cylinder approximation
- New `--fix-joints` argument converts specified joints to fixed
  (used to generate the legs-only training URDF)

Verified in IsaacGym viewer: all 28 links present and correctly
oriented.

Copy agibot_x1_train's `humanoid/` package as `asimov_rl/`, rename
all imports, and add Asimov-specific config/env:

- `algo/`, `utils/`, `envs/base/`, `scripts/` copied as-is
  (PPO, ActorCriticDH, state estimator, terrain, task registry)
- `envs/asimov/asimov_stand_config.py`: 12-DOF lower-body config
  - URDF: `asimov_v1_legs.urdf` (upper body + toes converted to
  - URDF: `asimov_v1_legs.urdf` (upper body + toes converted to
    fixed joints, yielding exactly 12 active DOF matching X1 layout)
    fixed joints, yielding exactly 12 active DOF matching X1 layout)
  - Init pose: pelvis at 0.66 m, hip pitch ±0.30, knee ±0.60,
  - Init pose: pelvis at 0.66 m, hip pitch ±0.30, knee ±0.60,
    ankle pitch -0.30
    ankle pitch -0.30
  - `base_height_target`: 0.58 m (vs X1 0.61 m)
  - `base_height_target`: 0.58 m (vs X1 0.61 m)
  - `foot_min_dist`: 0.15 m (Asimov hip width ~0.135 m)
  - `foot_min_dist`: 0.15 m (Asimov hip width ~0.135 m)
  - `terminate_after_contacts_on`: `pelvis_link`
  - `terminate_after_contacts_on`: `pelvis_link`
  - `foot_name`: "ankle_roll", `knee_name`: "knee"
  - `foot_name`: "ankle_roll", `knee_name`: "knee"
  - PD gains, domain randomization ranges copied from X1 as
  - PD gains, domain randomization ranges copied from X1 as
    starting point (to retune in Phase 0.4 with motor specs)
    starting point (to retune in Phase 0.4 with motor specs)
- `envs/asimov/asimov_stand_env.py`: thin adaptation of
- `envs/asimov/asimov_stand_env.py`: thin adaptation of
  X1DHStandEnv (reward functions, observation construction, and
  X1DHStandEnv (reward functions, observation construction, and
  swing-leg reference state all reused unchanged because the
  swing-leg reference state all reused unchanged because the
  12-DOF order matches X1)
  12-DOF order matches X1)
- `envs/__init__.py`: register `asimov_stand` task
- `envs/__init__.py`: register `asimov_stand` task
- `setup.py`: rename package, keep dependency list
- `setup.py`: rename package, keep dependency list

- `software/resources/robots/asimov_v1/urdf/asimov_v1.urdf`
  (27 joints — full body, for future stages)
- `software/resources/robots/asimov_v1/urdf/asimov_v1_legs.urdf`
  (12 active DOF — for Phase 1-2 training)
- `software/resources/robots/asimov_v1/meshes/*.STL` (28 files)
- `software/STAGE1_REPORT.md`: stage summary, validation steps,
  known risks

- Python syntax + import paths: all OK
- Config loads standalone: `num_actions=12`,
  `num_observations=3102`, all 12 default joint angles map to
  URDF joints
- IsaacGym viewer: full body visible with correct kinematic
  structure (verified by user screenshot)

File: software/resources/robots/asimov_v1/urdf/asimov_v1_legs.urdf (robot description, URDF)
Before this commit: robot asimov_v1, 28 links, 27 joints
Joints:
- joint left_elbow_joint: axis 0 -1 0 -> (none); limit lower=0 upper=2.44346 effort=200 velocity=20 -> (none); type revolute -> fixed
- joint left_shoulder_pitch_joint: axis 0 1 0 -> (none); limit lower=-3.14159 upper=0.872665 effort=200 velocity=20 -> (none); type revolute -> fixed
- joint left_shoulder_roll_joint: axis -1 0 0 -> (none); limit lower=-1.5708 upper=0 effort=200 velocity=20 -> (none); type revolute -> fixed
- joint left_shoulder_yaw_joint: axis 0 0 -1 -> (none); limit lower=-1.5708 upper=1.5708 effort=200 velocity=20 -> (none); type revolute -> fixed
- joint left_toe_joint: axis 0.010532 0.99994 0 -> (none); limit lower=-1.047 upper=0 effort=200 velocity=20 -> (none); type revolute -> fixed
- joint left_wrist_yaw_joint: axis 0.76604444 0 -0.64278761 -> (none); limit lower=-3.14159 upper=3.14159 effort=200 velocity=20 -> (none); type revolute -> fixed
- joint neck_pitch_joint: axis 0 1 0 -> (none); limit lower=-0.785398 upper=0.785398 effort=200 velocity=20 -> (none); type revolute -> fixed
- joint neck_yaw_joint: axis 0 0 1 -> (none); limit lower=-1.5708 upper=1.5708 effort=200 velocity=20 -> (none); type revolute -> fixed
- joint right_elbow_joint: axis 0 1 0 -> (none); limit lower=-2.44346 upper=0 effort=200 velocity=20 -> (none); type revolute -> fixed
- joint right_shoulder_pitch_joint: axis 0 -1 0 -> (none); limit lower=-0.872665 upper=3.14159 effort=200 velocity=20 -> (none); type revolute -> fixed
- joint right_shoulder_roll_joint: axis -1 0 0 -> (none); limit lower=0 upper=1.5708 effort=200 velocity=20 -> (none); type revolute -> fixed
- joint right_shoulder_yaw_joint: axis 0 0 -1 -> (none); limit lower=-1.5708 upper=1.5708 effort=200 velocity=20 -> (none); type revolute -> fixed
- joint right_toe_joint: axis 0.0074685 -0.99997 0 -> (none); limit lower=0 upper=1.047 effort=200 velocity=20 -> (none); type revolute -> fixed
- joint right_wrist_yaw_joint: axis 0.76604444 0 -0.64278761 -> (none); limit lower=-3.14159 upper=3.14159 effort=200 velocity=20 -> (none); type revolute -> fixed
- joint waist_yaw_joint: axis 0 0 1 -> (none); limit lower=-1.5708 upper=1.5708 effort=200 velocity=20 -> (none); type revolute -> fixed
