Commit message: Updating ankle roll joint range for URDF, too

File: sim-model/urdf/asimov_1.urdf (robot description, URDF)
Before this commit: robot asimov_1, 26 links, 25 joints
Joints:
- joint left_ankle_roll_joint: limit lower=-0.1 upper=0.1 effort=17 velocity=9.32 -> lower=-0.35 upper=0.35 effort=17 velocity=9.32
- joint right_ankle_roll_joint: limit lower=-0.1 upper=0.1 effort=17 velocity=9.32 -> lower=-0.35 upper=0.35 effort=17 velocity=9.32

Commit message: fix(sim-model): Update urdf and xml motion range to align with the hardware limits

File: sim-model/urdf/asimov_1.urdf (robot description, URDF)
Before this commit: robot asimov_1, 26 links, 25 joints
Joints:
- joint left_elbow_joint: limit lower=0 upper=2.443461 effort=12 velocity=9.32 -> lower=0 upper=2.0944 effort=12 velocity=9.32
- joint left_hip_pitch_joint: limit lower=-2.094395 upper=1 effort=45 velocity=12.57 -> lower=-1.57 upper=1.57 effort=45 velocity=12.57
- joint right_elbow_joint: limit lower=-2.443461 upper=0 effort=12 velocity=9.32 -> lower=-2.0944 upper=0 effort=12 velocity=9.32
- joint right_hip_pitch_joint: limit lower=-1 upper=2.094395 effort=45 velocity=12.57 -> lower=-1.57 upper=1.57 effort=45 velocity=12.57
